Commit message: added simplified model

File: urdf/era.urdf.xacro (robot description, xacro)
@@ -4,5 +4,5 @@
   <xacro:arg name="fixed" default="false"/>
   <xacro:arg name="robot_ns" default=""/>
-  <xacro:include filename="$(find era_description)/urdf/era.xacro"/>
+  <xacro:include filename="$(find era_description)/urdf/era2.xacro"/>
   <!-- <xacro:leo_erc_sim robot_ns="$(arg robot_ns)"
                      fixed="$(arg fixed)"/> -->

File: urdf/materials.xacro (robot description, xacro)
@@ -1,4 +1,4 @@
 <?xml version="1.0" ?>
-<robot name="era" xmlns:xacro="http://www.ros.org/wiki/xacro" >
+<robot name="era2" xmlns:xacro="http://www.ros.org/wiki/xacro" >
 <material name="silver_default">
   <color rgba="0.700 0.700 0.700 1.000"/>
@@ -13,6 +13,6 @@
   <color rgba="0.8156862745098039 0.8156862745098039 0.8156862745098039 1.0"/>
 </material>
-<material name="opaque144144144">
-  <color rgba="0.5647058823529412 0.5647058823529412 0.5647058823529412 1.0"/>
+<material name="opaque161616">
+  <color rgba="0.06274509803921569 0.06274509803921569 0.06274509803921569 1.0"/>
 </material>
 </robot>
